File: SplashPad.kicad_pcb (KiCad board)
At the start: 2 copper layers, 100 x 100 mm, 35 parts, among them SW1 SW_Push_45deg, SW10 RotaryEncoder_Switch, SW11 RotaryEncoder_Switch, SW2 SW_Push_45deg, SW3 SW_Push_45deg, SW4 SW_Push_45deg, SW5 SW_Push_45deg, SW6 SW_Push_45deg, SW7 SW_Push_45deg, SW8 SW_Push_45deg, SW9 SW_Push_45deg

Commit message: fine tuning
Parts:
- removed XIAO HERE: XIAO-RP2040-DIP, Seeed Studio XIAO Series Library:XIAO-RP2040-DIP
- added REF**: 3.2mm_M3, MountingHole:MountingHole_3.2mm_M3, F.Cu at (136.5, 146.0)
- added REF**: 3.2mm_M3, MountingHole:MountingHole_3.2mm_M3, F.Cu at (196.5, 146.0)
- added REF**: 3.2mm_M3, MountingHole:MountingHole_3.2mm_M3, F.Cu at (136.5, 70.0)
- added REF**: 3.2mm_M3, MountingHole:MountingHole_3.2mm_M3, F.Cu at (196.5, 70.0)
- added U1: XIAO-RP2040-DIP, Seeed Studio XIAO Series Library:XIAO-RP2040-DIP, F.Cu at (166.5, 77.4)
- moved D23 1.00 mm to (185.8, 70.5)
- moved SW11 1.00 mm to (178.2, 78.0)
Other:
- board size 100 x 100 mm -> 67 x 83 mm
- board text added: "XIAO HERE"

Commit message: The Fun Part
Parts:
- renumbered REF** to HOLE1, REF** to HOLE2, REF** to HOLE3, REF** to HOLE4
Routing:
- net +3.3V: track 0.00 -> 336.5 mm, vias 0 -> 3
- net GND: track 0.00 -> 323.0 mm, vias 0 -> 1
- net Row 2: track 0.00 -> 120.6 mm, vias 0 -> 2
- net Column 2: track 0.00 -> 106.6 mm, vias 0 -> 3
- net Row 1: track 0.00 -> 88.9 mm
- net Net-(D7-A): track 0.00 -> 80.8 mm, vias 0 -> 2
- net Row 0: track 0.00 -> 75.0 mm
- net Column 1: track 0.00 -> 72.8 mm
- net Net-(D3-A): track 0.00 -> 68.5 mm, vias 0 -> 1
- net Column 0: track 0.00 -> 56.0 mm
- net Net-(D8-A): track 0.00 -> 39.7 mm, vias 0 -> 1
- net Net-(D4-A): track 0.00 -> 39.7 mm, vias 0 -> 1
- net LED Data: track 0.00 -> 38.5 mm, vias 0 -> 1
- net Pot Button 2: track 0.00 -> 36.1 mm
- net Net-(D6-A): track 0.00 -> 33.8 mm, vias 0 -> 1
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
Commit message: encoder fix
Parts:
- removed the SW10 at (139.8, 78.0)
- renumbered SW11 to SW10
Connections:
- U1 pad 4: Pot Button 2 -> unconnected-(U1-GPIO29/ADC3/A3-Pad4)
Routing:
- net Row 2: track 120.6 -> 41.1 mm, vias 2 -> 0
- net Pot Button 2: track 36.1 -> 0.00 mm
- net +3.3V: track 336.5 -> 311.9 mm, vias 3 -> 4
- net Pot Analog 1: track 25.4 -> 0.84 mm
- net Column 2: track 106.6 -> 93.8 mm, vias 3 -> 1
- net Net-(D7-A): track 80.8 -> 87.4 mm, vias 2 -> 1
- net Pot Button 1: track 5.89 -> 0.84 mm
- net Net-(D4-A): track 39.7 -> 44.3 mm
- net Net-(D8-A): track 39.7 -> 36.1 mm, vias 1 -> 0
- net Row 1: track 88.9 -> 85.5 mm
- net Row 0: track 75.0 -> 71.7 mm
- net GND: track 323.0 -> 319.9 mm
- net Pot Analog 2: track 25.4 -> 23.6 mm, vias 1 -> 0
- net Net-(D3-A): track 68.5 -> 66.8 mm
- net Net-(D2-A): track 29.9 -> 31.1 mm, vias 0 -> 1
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
Commit message: trace fix
Routing:
- net Row 2: track 41.1 -> 150.8 mm

Commit message: Awesome Silkscreen Art!
Parts:
- added G***: LOGO, LOGO, F.Cu at (155.5, 146.5)
- added G***: LOGO, LOGO, B.Cu at (186.0, 77.0)
- added G***: LOGO, LOGO, B.Cu at (194.5, 135.5)
- added G***: LOGO, LOGO, B.Cu at (182.0, 143.5)
- added G***: LOGO, LOGO, B.Cu at (176.5, 101.5)
- added G***: LOGO, LOGO, B.Cu at (166.5, 70.0)
- added G***: LOGO, LOGO, B.Cu at (138.5, 82.9)
- added G***: LOGO, LOGO, B.Cu at (148.5, 73.0)
- added G***: LOGO, LOGO, B.Cu at (177.0, 132.5)
- added G***: LOGO, LOGO, B.Cu at (186.9, 126.1)
- added G***: OrpheusHackClubIcon, SKS:OrpheusHackClubIcon, B.Cu at (149.1, 91.0)
- added G***: LOGO, LOGO, F.Cu at (166.5, 70.0)
- added G***: LOGO, LOGO, B.Cu at (194.5, 93.0)
- added G***: LOGO, LOGO, F.Cu at (139.0, 80.5)
- added G***: LOGO, LOGO, F.Cu at (179.5, 70.0)
- added G***: LOGO, LOGO, F.Cu at (149.5, 80.0)
- added G***: LOGO, LOGO, B.Cu at (176.5, 120.5)
- added G***: LOGO, LOGO, B.Cu at (151.0, 133.5)
- added G***: LOGO, LOGO, B.Cu at (162.5, 81.5)
- added G***: LOGO, LOGO, B.Cu at (141.0, 115.0)
Other:
- board text added: "@SharKingStudios"
